File: Shark50.kicad_pcb (KiCad board)
At the start: 2 copper layers, 24 parts, among them J1 USB_B_Mini, SW1 MXSwitch, SW2 MXSwitch, SW3 MXSwitch, SW4 MXSwitch, U1 ATmega32U4-AU, Y1 16Mhz

Commit message: matrix done
Parts:
- added D10: 1N4148W, Diode_SMD:D_SOD-123, B.Cu at (204.3, -11.2)
- added D11: 1N4148W, Diode_SMD:D_SOD-123, B.Cu at (210.0, -11.2)
- added D12: 1N4148W, Diode_SMD:D_SOD-123, B.Cu at (192.8, -14.6)
- added D13: 1N4148W, Diode_SMD:D_SOD-123, B.Cu at (198.5, -14.6)
- added D14: 1N4148W, Diode_SMD:D_SOD-123, B.Cu at (210.0, -14.6)
- added D15: 1N4148W, Diode_SMD:D_SOD-123, B.Cu at (204.3, -17.9)
- added D16: 1N4148W, Diode_SMD:D_SOD-123, B.Cu at (204.3, -14.6)
- added D17: 1N4148W, Diode_SMD:D_SOD-123, B.Cu at (224.3, 15.6)
- added D18: 1N4148W, Diode_SMD:D_SOD-123, B.Cu at (224.3, 12.3)
- added D19: 1N4148W, Diode_SMD:D_SOD-123, B.Cu at (218.6, 8.94)
- added D20: 1N4148W, Diode_SMD:D_SOD-123, B.Cu at (224.3, 8.94)
- added D21: 1N4148W, Diode_SMD:D_SOD-123, B.Cu at (218.6, 5.59)
- added D22: 1N4148W, Diode_SMD:D_SOD-123, B.Cu at (224.3, 5.59)
- added D23: 1N4148W, Diode_SMD:D_SOD-123, B.Cu at (218.6, 2.24)
- added D24: 1N4148W, Diode_SMD:D_SOD-123, B.Cu at (224.3, 2.24)
- added D25: 1N4148W, Diode_SMD:D_SOD-123, B.Cu at (192.8, -17.9)
- added D26: 1N4148W, Diode_SMD:D_SOD-123, B.Cu at (302.9, 76.1)
- added D27: 1N4148W, Diode_SMD:D_SOD-123, B.Cu at (297.2, 72.7)
- added D28: 1N4148W, Diode_SMD:D_SOD-123, B.Cu at (297.2, 69.4)
- added D29: 1N4148W, Diode_SMD:D_SOD-123, B.Cu at (291.4, 66.0)
- added D3: 1N4148W, Diode_SMD:D_SOD-123, B.Cu at (297.2, 66.0)
- added D30: 1N4148W, Diode_SMD:D_SOD-123, B.Cu at (285.7, 62.7)
- added D31: 1N4148W, Diode_SMD:D_SOD-123, B.Cu at (291.4, 62.7)
- added D32: 1N4148W, Diode_SMD:D_SOD-123, B.Cu at (308.7, 76.0)
- added D33: 1N4148W, Diode_SMD:D_SOD-123, B.Cu at (302.9, 72.7)
- added D34: 1N4148W, Diode_SMD:D_SOD-123, B.Cu at (302.9, 69.4)
- added D35: 1N4148W, Diode_SMD:D_SOD-123, B.Cu at (314.4, 66.0)
- added D36: 1N4148W, Diode_SMD:D_SOD-123, B.Cu at (302.9, 66.0)
- added D37: 1N4148W, Diode_SMD:D_SOD-123, B.Cu at (308.7, 72.7)
- added D38: 1N4148W, Diode_SMD:D_SOD-123, B.Cu at (297.2, 62.7)
- added D39: 1N4148W, Diode_SMD:D_SOD-123, B.Cu at (314.4, 76.0)
- added D4: 1N4148W, Diode_SMD:D_SOD-123, B.Cu at (198.5, -17.9)
- added D40: 1N4148W, Diode_SMD:D_SOD-123, B.Cu at (302.9, 62.7)
- added D41: 1N4148W, Diode_SMD:D_SOD-123, B.Cu at (314.4, 72.7)
- added D42: 1N4148W, Diode_SMD:D_SOD-123, B.Cu at (308.7, 69.3)
- added D43: 1N4148W, Diode_SMD:D_SOD-123, B.Cu at (210.0, -17.9)
- added D44: 1N4148W, Diode_SMD:D_SOD-123, B.Cu at (314.4, 69.3)
- added D45: 1N4148W, Diode_SMD:D_SOD-123, B.Cu at (308.7, 66.0)
- added D5: 1N4148W, Diode_SMD:D_SOD-123, B.Cu at (204.3, -4.51)
- added D6: 1N4148W, Diode_SMD:D_SOD-123, B.Cu at (210.0, -4.51)
- added D7: 1N4148W, Diode_SMD:D_SOD-123, B.Cu at (204.3, -7.86)
- added D8: 1N4148W, Diode_SMD:D_SOD-123, B.Cu at (210.0, -7.86)
- added D9: 1N4148W, Diode_SMD:D_SOD-123, B.Cu at (198.5, -11.2)
- added R1: R_Small, Resistor_SMD:R_1206_3216Metric_Pad1.42x1.75mm_HandSolder, B.Cu at (314.3, 62.7)
- added SW10: O, acheron_MX:MX100, B.Cu at (128.6, -95.2)
- added SW11: P, acheron_MX:MX100, B.Cu at (147.6, -95.2)
- added SW12: [, acheron_MX:MX100, B.Cu at (166.7, -95.2)
- added SW13: ], acheron_MX:MX100, B.Cu at (185.7, -95.2)
- added SW14: BS, acheron_MX:MX100, B.Cu at (204.8, -95.2)
- added SW15: Tab_125, acheron_MX:MX125, B.Cu at (-40.5, -76.2)
- added SW16: LShift_175, acheron_MX:MX175, B.Cu at (-35.7, -57.1)
- added SW17: LCtrl_125, acheron_MX:MX125, B.Cu at (-40.5, -38.1)
- added SW18: A, acheron_MX:MX100, B.Cu at (-19.1, -76.2)
- added SW19: Z, acheron_MX:MX100, B.Cu at (-9.53, -57.1)
- added SW20: S, acheron_MX:MX100, B.Cu at (0.00, -76.2)
- added SW21: X, acheron_MX:MX100, B.Cu at (9.53, -57.1)
- added SW22: LAlt_125, acheron_MX:MX125, B.Cu at (2.38, -38.1)
- added SW23: D, acheron_MX:MX100, B.Cu at (19.1, -76.2)
- added SW24: C, acheron_MX:MX100, B.Cu at (28.6, -57.1)
- added SW25: F, acheron_MX:MX100, B.Cu at (38.1, -76.2)
- added SW26: V, acheron_MX:MX100, B.Cu at (47.6, -57.1)
- added SW27: Spc_700, acheron_MX:MX700, B.Cu at (81.0, -38.1)
- added SW28: G, acheron_MX:MX100, B.Cu at (57.1, -76.2)
- added SW29: B, acheron_MX:MX100, B.Cu at (66.7, -57.1)
- added SW30: H, acheron_MX:MX100, B.Cu at (76.2, -76.2)
- added SW31: N, acheron_MX:MX100, B.Cu at (85.7, -57.1)
- added SW32: J, acheron_MX:MX100, B.Cu at (95.2, -76.2)
- added SW33: M, acheron_MX:MX100, B.Cu at (104.8, -57.1)
- added SW34: K, acheron_MX:MX100, B.Cu at (114.3, -76.2)
- added SW35: <, acheron_MX:MX100, B.Cu at (123.8, -57.1)
- added SW36: L, acheron_MX:MX100, B.Cu at (133.3, -76.2)
- added SW37: >, acheron_MX:MX100, B.Cu at (142.9, -57.1)
- added SW38: :, acheron_MX:MX100, B.Cu at (152.4, -76.2)
- added SW39: ?, acheron_MX:MX100, B.Cu at (161.9, -57.1)
- added SW40: RAlt_125, acheron_MX:MX125, B.Cu at (159.5, -38.1)
- added SW41: ", acheron_MX:MX100, B.Cu at (171.4, -76.2)
- added SW42: RShift_125, acheron_MX:MX125, B.Cu at (183.4, -57.1)
- added SW43: Ent_175, acheron_MX:MX175, B.Cu at (197.6, -76.2)
- added SW44: Fn, acheron_MX:MX100, B.Cu at (204.8, -57.1)
- added SW45: RCtrl_125, acheron_MX:MX125, B.Cu at (202.4, -38.1)
- added SW5: R, acheron_MX:MX100, B.Cu at (33.3, -95.2)
- added SW6: T, acheron_MX:MX100, B.Cu at (52.4, -95.2)
- added SW7: Y, acheron_MX:MX100, B.Cu at (71.4, -95.2)
- added SW8: U, acheron_MX:MX100, B.Cu at (90.5, -95.2)
- added SW9: I, acheron_MX:MX100, B.Cu at (109.5, -95.2)
- C1: renamed from C5; moved to B.Cu
- C2: renamed from C4; moved to B.Cu
- C3: renamed from C6; moved to B.Cu
- C4: renamed from C7; moved to B.Cu
- C5: renamed from C2; moved to B.Cu
- C6: renamed from C3; moved to B.Cu
- C7: renamed from C8; moved to B.Cu
- C8: renamed from C1; moved to B.Cu
- D1, D2: value D_Small -> 1N4148W; moved to B.Cu
- D3, D4, SWP1, U1, Y1: moved to B.Cu
- R2: renamed from R3; moved to B.Cu
- R3: renamed from R1; moved to B.Cu
- R4: renamed from R2; moved to B.Cu
- R5: renamed from R4; value 10k -> 1k; moved to B.Cu
- SW1: value MXSwitch -> Esc; moved to B.Cu
- SW2: value MXSwitch -> Q; moved to B.Cu
- SW3: value MXSwitch -> W; moved to B.Cu
- SW4: value MXSwitch -> E; moved to B.Cu
- moved R4 300.6 mm to (378.2, 78.9), turned to 180 degrees
- moved R3 288.7 mm to (372.2, 78.9), turned to 180 degrees
- moved R2 276.8 mm to (366.3, 78.9), turned to 180 degrees
- moved C4 265.1 mm to (372.8, 5.61), turned to 180 degrees
- moved R5 264.9 mm to (360.4, 78.9), turned to 180 degrees
- moved D1 264.1 mm to (372.3, 2.46), turned to 180 degrees
- moved SWP1 260.5 mm to (370.4, -2.59), turned to 180 degrees
- moved Y1 259.8 mm to (370.0, -8.39), turned to 180 degrees
- moved U1 255.7 mm to (367.9, -18.0), turned to 180 degrees
- moved D3 253.2 mm to (354.5, 78.9), turned to 180 degrees
- moved C5 246.7 mm to (363.2, -4.49), turned to 180 degrees
- moved C6 245.4 mm to (362.5, -8.93), turned to 180 degrees
- moved C8 242.7 mm to (349.2, 78.7), turned to 180 degrees
- moved D4 236.4 mm to (357.8, -12.1), turned to 180 degrees
- moved C3 236.3 mm to (357.8, -8.93), turned to 180 degrees
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Connections:
- C2 pad 1: GND -> Net-(C2-Pad1)
- R5 pad 1: GND -> Net-(R5-Pad1)
- SW3 pad 1: Col1 -> Col3
- SW4 pad 1: Col2 -> Col4
- SWP1 pad 1: GND -> Net-(C2-Pad1)
