File: Shark50.sch (KiCad schematic (older format))
At the start: 45 parts, among them J1 USB_B_Mini, SW1 Esc, SW10 O, SW11 P, SW12 [, SW13 ], SW14 BS, SW2 Q, SW3 W, SW4 E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

Commit message: last row
Parts:
- added D? (x31): 1N4148W, Diode_SMD:D_SOD-123, symbol Device:D_Small
- added SW?: Tab, acheron_MX:MX100, symbol acheronSymbols:MXSwitch
- added SW?: A, acheron_MX:MX100, symbol acheronSymbols:MXSwitch
- added SW?: S, acheron_MX:MX100, symbol acheronSymbols:MXSwitch
- added SW?: D, acheron_MX:MX100, symbol acheronSymbols:MXSwitch
- added SW?: F, acheron_MX:MX100, symbol acheronSymbols:MXSwitch
- added SW?: G, acheron_MX:MX100, symbol acheronSymbols:MXSwitch
- added SW?: H, acheron_MX:MX100, symbol acheronSymbols:MXSwitch
- added SW?: J, acheron_MX:MX100, symbol acheronSymbols:MXSwitch
- added SW?: K, acheron_MX:MX100, symbol acheronSymbols:MXSwitch
- added SW?: L, acheron_MX:MX100, symbol acheronSymbols:MXSwitch
- added SW?: :, acheron_MX:MX100, symbol acheronSymbols:MXSwitch
- added SW?: \", acheron_MX:MX100, symbol acheronSymbols:MXSwitch
- added SW?: Ent, acheron_MX:MX100, symbol acheronSymbols:MXSwitch
- added SW?: LShift, acheron_MX:MX100, symbol acheronSymbols:MXSwitch
- added SW?: Z, acheron_MX:MX100, symbol acheronSymbols:MXSwitch
- added SW?: X, acheron_MX:MX100, symbol acheronSymbols:MXSwitch
- added SW?: C, acheron_MX:MX100, symbol acheronSymbols:MXSwitch
- added SW?: V, acheron_MX:MX100, symbol acheronSymbols:MXSwitch
- added SW?: B, acheron_MX:MX100, symbol acheronSymbols:MXSwitch
- added SW?: N, acheron_MX:MX100, symbol acheronSymbols:MXSwitch
- added SW?: M, acheron_MX:MX100, symbol acheronSymbols:MXSwitch
- added SW?: <, acheron_MX:MX100, symbol acheronSymbols:MXSwitch
- added SW?: >, acheron_MX:MX100, symbol acheronSymbols:MXSwitch
- added SW?: ?, acheron_MX:MX100, symbol acheronSymbols:MXSwitch
- added SW?: RShift, acheron_MX:MX100, symbol acheronSymbols:MXSwitch
- added SW?: Fn, Fn, symbol acheronSymbols:MXSwitch
- added SW?: LCtrl, acheron_MX:MX100, symbol acheronSymbols:MXSwitch
- added SW?: LAlt, acheron_MX:MX100, symbol acheronSymbols:MXSwitch
- added SW?: Spc, acheron_MX:MX100, symbol acheronSymbols:MXSwitch
- added SW?: RAlt, acheron_MX:MX100, symbol acheronSymbols:MXSwitch
- added SW?: RCtrl, acheron_MX:MX100, symbol acheronSymbols:MXSwitch
Connections:
- net labels added: Row2, Row3
- wire segments 124 -> 232

Commit message: matrix done
Connections:
- net Row4: now reaches D?.1 (K), D?.1 (K), D?.1 (K), D?.1 (K), D?.1 (K)
Changed lines of the file:
@@
 	17150 5250 17150 6700
-Wire Wire Line
-	4800 5800 5850 5800
-Connection ~ 5850 5800
 Wire Wire Line
 	5850 5800 7950 5800
@@
 Wire Wire Line
 	15750 5800 17600 5800
+Wire Wire Line
+	5850 5800 5100 5800
+Connection ~ 5850 5800
+Text GLabel 5100 5800 0    50   Input ~ 0
+Row4
 $EndSCHEMATC

Commit message: matrix done
Parts:
- R1: footprint (none) -> Resistor_SMD:R_1206_3216Metric_Pad1.42x1.75mm_HandSolder
- SW15: renamed from SW?; value Tab -> Tab_125; footprint acheron_MX:MX100 -> acheron_MX:MX125
- SW16: renamed from SW?; value LShift -> LShift_175; footprint acheron_MX:MX100 -> acheron_MX:MX175
- SW17: renamed from SW?; value LCtrl -> LCtrl_125; footprint acheron_MX:MX100 -> acheron_MX:MX125
- SW22: renamed from SW?; value LAlt -> LAlt_125; footprint acheron_MX:MX100 -> acheron_MX:MX125
- SW27: renamed from SW?; value Spc -> Spc_700; footprint acheron_MX:MX100 -> acheron_MX:MX700
- SW40: renamed from SW?; value RAlt -> RAlt_125; footprint acheron_MX:MX100 -> acheron_MX:MX125
- SW42: renamed from SW?; value RShift -> RShift_125; footprint acheron_MX:MX100 -> acheron_MX:MX125
- SW43: renamed from SW?; value Ent -> Ent_175; footprint acheron_MX:MX100 -> acheron_MX:MX175
- SW44: renamed from SW?; footprint Fn -> acheron_MX:MX100
- SW45: renamed from SW?; value RCtrl -> RCtrl_125; footprint acheron_MX:MX100 -> acheron_MX:MX125
- gave numbers to parts that had none: 52
